File: bldc_driver.kicad_pcb (KiCad board)
At the start: 2 copper layers, 50 x 50 mm, 105 parts, among them IC1 AS5047D-ATSM, IC2 STSPIN32G4, J1 Conn_01x02_Pin, J2 ST-Link, J3 Conn_01x05_Pin, P1 USB_C_Plug_USB2.0, Q1 NMOS, Q2 NMOS, Q3 NMOS, Q4 NMOS, Q5 NMOS, Q6 NMOS, U1 NJW1933, U2 TCAN332, Y1 Crystal_GND24

Commit message: なんとなく配線できてきた
Parts:
- removed C18: 0.1u, Capacitor_SMD:C_0603_1608Metric_Pad1.08x0.95mm_HandSolder
- removed D3: MS110F, bdm:MS110F
- removed H5: MountingHole, MountingHole:MountingHole_3.2mm_M3
- removed R1: 4.32k, Resistor_SMD:R_0603_1608Metric_Pad0.98x0.95mm_HandSolder
- removed the R4 at (75.4, 68.0)
- C15, C16, C19, C20, C21, C22, C24, C25, C26, C27, C28, C29, C3, C30, C31, C34, C4, Q1, Q2, Q3, Q4, Q5, Q6, R10, R13, R14, R17, R18, R19, R20, R23, R27, R29, R3, R30, R31, R32, R33, R34, R36, R37, R38, R39, R7, R8, R9: moved to B.Cu
- H1, H2: value MountingHole_Pad -> MountingHole; footprint MountingHole:MountingHole_2.5mm_Pad_TopBottom -> MountingHole:MountingHole_3.2mm_M3
- IC2: footprint stspin32g4:QFN50P900X900X100-65N-D -> stspin32g4:QFN50P900X900X100-65N-D-padlong; moved to B.Cu
- J1: footprint Connector_JST:JST_XH_S2B-XH-A-1_1x02_P2.50mm_Horizontal -> Connector_PinHeader_2.54mm:PinHeader_1x02_P2.54mm_Vertical; moved to B.Cu
- J2: footprint Connector_PinHeader_1.27mm:PinHeader_2x05_P1.27mm_Vertical -> sam:PinHeader_2x05_P1.27mm_Vertical_big
- J3: footprint Connector_JST:JST_XH_S5B-XH-A_1x05_P2.50mm_Horizontal -> sam:PinHeader_1x05_P1.27mm_Vertical_big
- R2: value 4.32k -> 10k; moved to B.Cu
- Y1: footprint Crystal:Crystal_SMD_SeikoEpson_FA238V-4Pin_3.2x2.5mm_HandSoldering -> Crystal:Crystal_SMD_SeikoEpson_FA238V-4Pin_3.2x2.5mm; moved to B.Cu
- moved Q1 110.2 mm to (176.3, 56.8)
- moved C25 104.5 mm to (175.5, 63.8), turned to 180 degrees
- moved C31 103.6 mm to (178.8, 57.3), turned to -90 degrees
- moved J3 103.0 mm to (170.4, 88.8), turned to 180 degrees
- moved Q2 101.3 mm to (172.3, 53.6), turned to 180 degrees
- moved C22 99.9 mm to (168.9, 75.4)
- moved C28 99.1 mm to (169.3, 57.3), turned to -90 degrees
- moved C19 98.3 mm to (167.1, 68.8)
- moved C20 95.7 mm to (165.3, 67.1)
- moved C5 95.6 mm to (159.2, 79.9)
- moved R6 95.6 mm to (170.9, 68.7), turned to 180 degrees
- moved C3 95.6 mm to (157.6, 80.0), turned to 135 degrees
- moved R5 95.5 mm to (170.9, 70.9), turned to 180 degrees
- moved C26 94.9 mm to (166.0, 63.8), turned to 180 degrees
- moved C36 94.6 mm to (151.4, 58.0), turned to -90 degrees
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- renumbered R26 to R4
Connections:
- C23 pad 1: /ADC1_7 -> /ADC1_9
- C24 pad 1: /VDD -> /+3V3
- C32 pad 1: /ADC1_9 -> /ADC1_7
- P1 pad A4: /USB_POW -> unconnected-(P1-VBUS-PadA4)
- P1 pad A9: /USB_POW -> unconnected-(P1-VBUS-PadA4)
- P1 pad B4: /USB_POW -> unconnected-(P1-VBUS-PadA4)
- P1 pad B9: /USB_POW -> unconnected-(P1-VBUS-PadA4)
- R11 pad 2: /ADC1_7 -> /ADC1_9
- R12 pad 1: /ADC1_7 -> /ADC1_9
- R15 pad 2: /OP1_INP -> /OP3_INP
- R16 pad 1: /OP1_INP -> /OP3_INP
- R2 pad 1: Net-(R1-Pad1) -> /+5V
- R24 pad 2: /OP3_INP -> /OP1_INP
- R25 pad 1: /OP3_INP -> /OP1_INP
- R35 pad 2: /ADC1_9 -> /ADC1_7
- R7 pad 1: /VDD -> /+3V3
Routing:
- net GND: track 0.00 -> 101.0 mm, vias 0 -> 65
- net /+3V3: track 0.00 -> 70.9 mm, vias 0 -> 5
- net +48V: track 0.00 -> 62.3 mm, vias 0 -> 59
- net /+5V: track 0.00 -> 34.0 mm, vias 0 -> 1
- net /FDCAN1_TX: track 0.00 -> 32.0 mm, vias 0 -> 2
- net /+3V3A: track 0.00 -> 31.3 mm, vias 0 -> 1
- net /W: track 0.00 -> 28.4 mm, vias 0 -> 2
- net /FDCAN1_RX: track 0.00 -> 27.0 mm, vias 0 -> 2
- net /SHUNT_U: track 0.00 -> 25.7 mm, vias 0 -> 1
- net /SHUNT_W: track 0.00 -> 24.9 mm, vias 0 -> 2
- net /HALL_U: track 0.00 -> 23.9 mm, vias 0 -> 1
- net Net-(Q1-G): track 0.00 -> 23.7 mm
- net /LD2: track 0.00 -> 23.5 mm, vias 0 -> 2
- net /SHUNT_V: track 0.00 -> 22.4 mm, vias 0 -> 2
- net /LD1: track 0.00 -> 22.2 mm, vias 0 -> 2
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- added copper zone on B.Cu, net +48V
- added copper zone on F.Cu, net +48V
- added copper zone on In1.Cu, net +48V
- added copper zone on B.Cu, net /SHUNT_U
- added copper zone on B.Cu, net /SHUNT_V
- added copper zone on B.Cu, net /SHUNT_W
- added copper zone on B.Cu, net /U
- added copper zone on B.Cu, net /V
- added copper zone on B.Cu, net /W
- added copper zone on B.Cu, net GND
- added copper zone on F.Cu, net GND
- added copper zone on In1.Cu, net GND
- added copper zone on In2.Cu, net GND
Other:
- board size 50 x 50 mm -> 35 x 45 mm
- copper layers 2 -> 4

Commit message: 配線がほとんど終わった
Parts:
- moved R9 10.3 mm to (154.1, 91.2)
- moved R13 10.3 mm to (155.7, 91.2)
- moved R10 10.2 mm to (157.4, 91.2)
- moved R14 9.97 mm to (159.0, 91.2)
- moved J3 6.11 mm to (166.0, 93.0), turned to 90 degrees
- moved J2 4.08 mm to (169.4, 85.1), turned to 0 degrees
- moved C15 0.83 mm to (161.7, 91.8)
- moved R3 0.74 mm to (165.2, 90.3)
- moved R2 0.63 mm to (161.8, 90.3)
- moved R5 0.26 mm to (170.9, 70.6)
- moved U2 0.25 mm to (148.3, 71.8)
- moved C17 0.13 mm to (159.0, 85.0)
Connections:
- J3 pad 3: /HALL_U -> /HALL_W
- J3 pad 5: /HALL_W -> /HALL_U
Routing:
- net Net-(D4-A): track 1.35 -> 16.4 mm
- net Net-(D6-A): track 1.93 -> 14.9 mm, vias 1 -> 2
- net Net-(D5-A): track 2.10 -> 14.8 mm, vias 1 -> 2
- net Net-(D7-A): track 3.26 -> 14.7 mm, vias 1 -> 2
- net /HALL_W: track 15.3 -> 26.6 mm
- net /LD4: track 14.1 -> 24.5 mm
- net /HALL_V: track 21.4 -> 30.8 mm
- net /HALL_U: track 23.9 -> 32.0 mm
- net /LD2: track 23.5 -> 17.1 mm
- net GND: track 101.0 -> 105.9 mm, vias 65 -> 114
- net /LD1: track 22.2 -> 17.5 mm
- net /+3V3: track 70.9 -> 68.6 mm
- net /+5V: track 34.0 -> 36.1 mm
- net /SWDIO: track 15.2 -> 17.1 mm, vias 0 -> 1
- net /SWCLK: track 15.8 -> 16.8 mm, vias 1 -> 0
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- added copper zone on In2.Cu, net +48V

Commit message: ガーバー吐いた
Parts:
- added G***: LOGO, sam:loki_log, F.Cu at (169.0, 67.2)
- C15: value 220P -> 330p; footprint Capacitor_SMD:C_0402_1005Metric_Pad0.74x0.62mm_HandSolder -> Capacitor_SMD:C_0603_1608Metric_Pad1.08x0.95mm_HandSolder
- D1: value D -> RSX101VAM
- R5, R6: moved to B.Cu
- moved R5 6.60 mm to (177.4, 71.9), turned to 0 degrees
- moved R6 6.50 mm to (177.4, 68.8), turned to 0 degrees
- moved Q2 1.02 mm to (172.3, 54.6)
- moved Q4 1.02 mm to (162.8, 54.6)
- moved Q6 1.02 mm to (153.1, 54.6)
- moved R20 0.89 mm to (172.2, 58.0)
- moved R30 0.89 mm to (162.6, 58.0)
- moved R37 0.89 mm to (152.9, 58.0)
- moved C15 0.18 mm to (161.8, 91.9)
Routing:
- net GND: track 105.9 -> 104.4 mm, vias 114 -> 118
- net /W: track 28.4 -> 27.0 mm
- net Net-(P1-CC): track 2.71 -> 4.14 mm, vias 0 -> 1
- net Net-(Q4-G): track 11.1 -> 10.0 mm
- net Net-(Q6-G): track 11.5 -> 10.4 mm
- net Net-(Q2-G): track 10.3 -> 9.29 mm
- net /HALL_U: track 32.0 -> 31.0 mm
- net Net-(P1-VCONN): track 1.98 -> 2.87 mm, vias 0 -> 1
- net /HALL_V: track 30.8 -> 30.2 mm
Other:
- board text added: "+"
- board text added: "-"
- board text added: "5"
- board text added: "AS5047"
- board text added: "CAN"
- board text added: "G"
- board text added: "H"
- board text added: "L"
- board text added: "Loki"
- board text added: "ST-Link"
- board text added: "U"
- board text added: "V"
- board text added: "W"
- board text added: "stspin32g4"

Commit message: 値及びフットプリント修正
Parts:
- added C18: 220p, Capacitor_SMD:C_0402_1005Metric_Pad0.74x0.62mm_HandSolder, B.Cu at (161.7, 92.8)
- C10, C11, C7: footprint Capacitor_SMD:C_1206_3216Metric_Pad1.33x1.80mm_HandSolder -> Capacitor_SMD:C_0805_2012Metric_Pad1.18x1.45mm_HandSolder
- C15: value 330p -> 220p; footprint Capacitor_SMD:C_0603_1608Metric_Pad1.08x0.95mm_HandSolder -> Capacitor_SMD:C_0402_1005Metric_Pad0.74x0.62mm_HandSolder
- C25, C26, C27, C30, C32, C34: value 2.2n -> 1n
- C28, C29, C31: value 1u -> 0.1u
- D1: value RSX101VAM -> D
- moved C7 0.25 mm to (165.7, 88.6)
- moved C15 0.21 mm to (161.7, 91.7)
Routing:
- net /+5V: track 36.1 -> 37.2 mm
- net Net-(U1-FB): track 5.36 -> 6.44 mm
- net Net-(D5-A): track 14.8 -> 13.9 mm
- net Net-(D6-A): track 14.9 -> 14.0 mm
- net Net-(D7-A): track 14.7 -> 13.9 mm
