File: bldc_driver.kicad_pcb (KiCad board)
At the start: 4 copper layers, 35 x 45 mm, 102 parts, among them IC1 AS5047D-ATSM, IC2 STSPIN32G4, J1 Conn_01x02_Pin, J2 ST-Link, J3 Conn_01x05_Pin, P1 USB_C_Plug_USB2.0, Q1 NMOS, Q2 NMOS, Q3 NMOS, Q4 NMOS, Q5 NMOS, Q6 NMOS, U1 NJW1933, U2 TCAN332, Y1 Crystal_GND24

Commit message: QDD用に修正開始
Parts:
- removed C22: 0.1u, Capacitor_SMD:C_0603_1608Metric_Pad1.08x0.95mm_HandSolder
- removed H3: MountingHole, MountingHole:MountingHole_3.2mm_M3
- removed J3: Conn_01x05_Pin, sam:PinHeader_1x05_P1.27mm_Vertical_big
- removed P1: USB_C_Plug_USB2.0, Connector_USB:USB_C_Receptacle_XKB_U262-16XN-4BVC11
- removed R7: 22k, Resistor_SMD:R_0603_1608Metric_Pad0.98x0.95mm_HandSolder
- removed R8: 10k, Resistor_SMD:R_0603_1608Metric_Pad0.98x0.95mm_HandSolder
- added J4: USB_C_Receptacle_USB2.0_14P, Connector_USB:USB_C_Receptacle_XKB_U262-16XN-4BVC11, F.Cu at (177.4, 70.6)
- R10, R13, R14, R9: moved to F.Cu
- moved H2 18.2 mm to (154.0, 96.5)
- moved L1 11.1 mm to (167.6, 86.4), turned to 0 degrees
- moved J2 10.1 mm to (176.7, 78.0)
- moved R9 9.38 mm to (146.9, 85.1)
- moved R13 9.29 mm to (148.7, 85.1)
- moved R10 9.19 mm to (150.5, 85.1)
- moved R14 9.10 mm to (152.3, 85.1)
- moved H4 7.43 mm to (171.0, 96.5)
- moved C7 6.38 mm to (165.1, 95.0)
- moved H1 5.02 mm to (171.0, 79.5)
- moved C15 4.74 mm to (161.1, 96.4)
- moved D2 4.74 mm to (160.9, 98.3)
- moved R2 4.74 mm to (161.1, 95.0)
- moved R3 4.74 mm to (164.6, 95.0)
- moved U1 4.74 mm to (162.0, 95.0)
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Connections:
- IC2 pad 44: /HALL_W -> unconnected-(IC2-PA8-Pad44)
- IC2 pad 45: /HALL_V -> unconnected-(IC2-PA9-Pad45)
- IC2 pad 46: /HALL_U -> unconnected-(IC2-PA10-Pad46)
- IC2 pad 52: /SCREF -> /+3V3
Routing:
- net /HALL_U: track 31.0 -> 0.00 mm, vias 1 -> 0
- net /HALL_V: track 30.2 -> 0.00 mm, vias 1 -> 0
- net /HALL_W: track 26.6 -> 0.00 mm, vias 1 -> 0
- net /+3V3: track 68.6 -> 51.4 mm, vias 5 -> 3
- net /SW: track 17.4 -> 1.45 mm
- net Net-(D4-A): track 16.4 -> 1.77 mm, vias 1 -> 0
- net /+5V: track 37.2 -> 23.5 mm, vias 1 -> 2
- net Net-(D6-A): track 14.0 -> 1.82 mm, vias 2 -> 0
- net Net-(D5-A): track 13.9 -> 1.81 mm, vias 2 -> 0
- net Net-(D7-A): track 13.9 -> 1.82 mm, vias 2 -> 0
- net /VCC: track 20.6 -> 9.27 mm
- net /LD4: track 24.5 -> 13.4 mm
- net /FDCAN1_TX: track 32.0 -> 20.8 mm, vias 2 -> 1
- net (no net): track 0.00 -> 7.90 mm
- net unconnected-(P1-VBUS-PadA4): track 6.68 -> 0.00 mm
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Other:
- board size 35 x 45 mm -> 35 x 50 mm
- board text removed: "5"
- board text removed: "G"

Commit message: 修正完了
Parts:
- added G***: LOGO, phoenix-daughter-pcb:TRAPS_logo_trans_1000x1000, B.Cu at (150.2, 87.3)
- added J3: SPI_CON, Connector_PinHeader_2.54mm:PinHeader_2x03_P2.54mm_Vertical, F.Cu at (178.1, 88.5)
- moved J4 1.91 mm to (176.7, 79.9)
- moved G*** 0.90 mm to (168.9, 68.1)
- moved D1 0.25 mm to (166.6, 77.9)
- turned C10 to 180 degrees
- turned C11 to 180 degrees
- renumbered C18 to C16, C16 to C17, C17 to C18, C23 to C22, C24 to C23, C25 to C24, C26 to C25, C27 to C26, C28 to C27, C29 to C28, C30 to C29, C31 to C30, C32 to C31, C33 to C32, C34 to C33, C35 to C34, C36 to C35, D4 to D3, D5 to D4, D6 to D5, D7 to D6, H4 to H3, J4 to J1, J1 to J2, J2 to J4, R2 to R1, R14 to R10, R15 to R11, R16 to R12, R17 to R13, R18 to R14, R19 to R15, R20 to R16, R21 to R17, R22 to R18, R23 to R19, R3 to R2, R24 to R20, R25 to R21, R4 to R22, R27 to R23, R28 to R24, R29 to R25, R30 to R26, R31 to R27, R32 to R28, R33 to R29, R5 to R3, R34 to R30, R35 to R31, R36 to R32, R37 to R33, R38 to R34, R39 to R35, R6 to R4, R9 to R5, R10 to R6, R11 to R7, R12 to R8, R13 to R9
Routing:
- net /+3V3: track 51.4 -> 86.4 mm, vias 3 -> 5
- net /SPI1_CS: track 12.6 -> 26.2 mm
- net /SW: track 1.45 -> 13.9 mm
- net /SPI1_CLK: track 14.1 -> 25.8 mm
- net /VCC: track 9.27 -> 20.5 mm
- net /SPI1_MOSI: track 15.5 -> 24.9 mm
- net /SPI1_MISO: track 14.3 -> 23.2 mm
- net /FDCAN1_TX: track 20.8 -> 27.6 mm, vias 1 -> 2
- net /FDCAN1_RX: track 25.7 -> 31.8 mm, vias 1 -> 2
- net /GL_U: track 17.4 -> 13.5 mm
- net GND: track 103.7 -> 107.5 mm, vias 99 -> 153
- net +48V: track 62.3 -> 59.9 mm
- net /SWDIO: track 13.4 -> 15.0 mm
- net /SWCLK: track 16.0 -> 17.6 mm
- net /+3V3A: track 31.3 -> 29.8 mm
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Other:
- board text added: "+V"
- board text added: "CLK"
- board text added: "CS"
- board text added: "GND"
- board text added: "MISO"
- board text added: "MOSI"
