File: bldc_driver.kicad_sch (KiCad schematic)
At the start: 101 parts, among them IC1 AS5047D-ATSM, IC2 STSPIN32G4, J1 Conn_01x02_Pin, J3 Conn_01x05_Pin, J4 ST-Link, P1 USB_C_Plug_USB2.0, Q1 NMOS, Q2 NMOS, Q3 NMOS, Q4 NMOS, Q5 NMOS, Q6 NMOS, U1 NJW1933, U2 TCAN332, Y201 Crystal_GND24

Commit message: QDD用に修正開始
Parts:
- removed C22: 0.1u, Capacitor_SMD:C_0603_1608Metric_Pad1.08x0.95mm_HandSolder, symbol Device:C
- removed J3: Conn_01x05_Pin, sam:PinHeader_1x05_P1.27mm_Vertical_big, symbol Connector:Conn_01x05_Pin
- removed P1: USB_C_Plug_USB2.0, Connector_USB:USB_C_Receptacle_XKB_U262-16XN-4BVC11, symbol Connector:USB_C_Plug_USB2.0
- removed R7: 22k, Resistor_SMD:R_0603_1608Metric_Pad0.98x0.95mm_HandSolder, symbol Device:R
- removed R8: 10k, Resistor_SMD:R_0603_1608Metric_Pad0.98x0.95mm_HandSolder, symbol Device:R
- added J4: USB_C_Receptacle_USB2.0_14P, Connector_USB:USB_C_Receptacle_XKB_U262-16XN-4BVC11, symbol Connector:USB_C_Receptacle_USB2.0_14P
- renumbered J4 to J2, Y201 to Y1
Connections:
- net SCREF is gone; now on net +3V3: IC2.52 (SCREF)
- net GND: now also J4.A1 (GND), J4.A12 (GND), J4.B1 (GND), J4.B12 (GND), J4.S1 (SHIELD)
- net USB_DM: now also J4.A7 (D-), J4.B7 (D-)
- net USB_DP: now also J4.A6 (D+), J4.B6 (D+)
- net at R6.1: now also J4.B5 (CC2)
- net at R5.1: now also J4.A5 (CC1)
- net HALL_U: no longer names the net of IC2.46 (PA10)
- net HALL_V: no longer names the net of IC2.45 (PA9)
- net HALL_W: no longer names the net of IC2.44 (PA8)
- new net: J4.A4 (VBUS), J4.A9 (VBUS), J4.B4 (VBUS), J4.B9 (VBUS)
- no-connect marks 17 -> 20

Commit message: 修正完了
Parts:
- removed H3: MountingHole, MountingHole:MountingHole_3.2mm_M3, symbol Mechanical:MountingHole
- added J3: SPI_CON, Connector_PinHeader_2.54mm:PinHeader_2x03_P2.54mm_Vertical, symbol Connector_Generic:Conn_02x03_Odd_Even
- renumbered C18 to C16, C16 to C17, C17 to C18, C23 to C22, C24 to C23, C25 to C24, C26 to C25, C27 to C26, C28 to C27, C29 to C28, C30 to C29, C31 to C30, C32 to C31, C33 to C32, C34 to C33, C35 to C34, C36 to C35, D4 to D3, D5 to D4, D6 to D5, D7 to D6, H4 to H3, J4 to J1, J1 to J2, J2 to J4, R2 to R1, R14 to R10, R15 to R11, R16 to R12, R17 to R13, R18 to R14, R19 to R15, R20 to R16, R21 to R17, R22 to R18, R23 to R19, R3 to R2, R24 to R20, R25 to R21, R4 to R22, R27 to R23, R28 to R24, R29 to R25, R30 to R26, R31 to R27, R32 to R28, R33 to R29, R5 to R3, R34 to R30, R35 to R31, R36 to R32, R37 to R33, R38 to R34, R39 to R35, R6 to R4, R9 to R5, R10 to R6, R11 to R7, R12 to R8, R13 to R9
Connections:
- net +3V3: now also J3.2 (Pin_2)
- net GND: now also J3.4 (Pin_4)
- net SPI1_CLK: now also J3.3 (Pin_3)
- net SPI1_CS: now also J3.1 (Pin_1)
- net SPI1_MISO: now also J3.5 (Pin_5)
- net SPI1_MOSI: now also J3.6 (Pin_6)
Other:
- moved on the sheet: H3
